File: irrigation.kicad_pcb (KiCad board)
At the start: 2 copper layers, 57.3 x 46.3 mm, 43 parts, among them J1 - 12V +, J2 + Pump 1 -, J3 + Pump 2 -, J4 USB_C_Receptacle_USB2.0, J5 Water Level, Q1 IRF7401, Q2 IRF7401, SW1 Reset, SW2 Boot, U1 TPS5430DDA, U2 AMS1117-3.3, U3 SRV05-4, U4 ESP32-C3-WROOM-02

Commit message: Various bug fixes & improvements
Parts:
- added D6: LED, LED_SMD:LED_0603_1608Metric, F.Cu at (116.2, 52.6)
- added D7: LED, LED_SMD:LED_0603_1608Metric, F.Cu at (131.7, 56.0)
- added R3: 1k, Resistor_SMD:R_0603_1608Metric, F.Cu at (120.3, 52.6)
- added R4: 47k, Resistor_SMD:R_0603_1608Metric, F.Cu at (115.4, 55.9)
- added R5: 47k, Resistor_SMD:R_0603_1608Metric, F.Cu at (124.0, 56.0)
- added R6: 1k, Resistor_SMD:R_0603_1608Metric, F.Cu at (133.7, 56.0)
- added R9: 10k, Resistor_SMD:R_0603_1608Metric, F.Cu at (141.1, 59.1)
- C5: footprint Capacitor_SMD:CP_Elec_5x5.8 -> Capacitor_SMD:CP_Elec_6.3x7.7
- J1: value - 12V + -> - 12V +
- J2: value + Pump 1 - -> - Pump 1 +
- J3: value + Pump 2 - -> - Pump 2 +
- U4: footprint Espressif:ESP32-C3-WROOM-02 -> PCM_Espressif:ESP32-C3-WROOM-02
- moved R11 4.41 mm to (124.0, 60.4)
- moved R10 4.31 mm to (115.4, 60.3)
- moved D8 1.91 mm to (118.4, 65.5), turned to 180 degrees
- moved D9 1.30 mm to (128.0, 65.5), turned to 180 degrees
- moved J3 1.12 mm to (127.2, 76.2), turned to 180 degrees
- moved D5 1.10 mm to (142.6, 50.5)
- moved J2 0.91 mm to (116.2, 76.2), turned to 180 degrees
- moved SW2 0.88 mm to (145.7, 61.0)
- moved C3 0.83 mm to (121.8, 48.5)
- moved C5 0.82 mm to (148.6, 52.1)
- moved J1 0.67 mm to (117.0, 39.9), turned to 0 degrees
- moved C4 0.63 mm to (137.7, 52.1)
- moved Q1 0.61 mm to (119.2, 58.1)
- moved C6 0.35 mm to (159.8, 58.2)
- moved C7 0.35 mm to (163.4, 58.2)
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- renumbered D8 to D10, D6 to D8, D7 to D9, R3 to R10, R4 to R11, R7 to R12, R8 to R13, R9 to R14, R10 to R15, R11 to R16, R5 to R7, R6 to R8
Connections:
- SW2 pad 1: GND -> Net-(R7-Pad1)
- SW2 pad 2: GND -> Net-(R7-Pad1)
Routing:
- net +12V: track 92.9 -> 108.1 mm
- net /GPIO5: track 51.9 -> 61.4 mm, vias 0 -> 4
- net Net-(R7-Pad1): track 0.00 -> 6.80 mm
- net Net-(J1-Pin_1): track 7.30 -> 14.0 mm
- net /GPIO6: track 41.8 -> 45.3 mm, vias 0 -> 2
- net +3V3: track 45.9 -> 48.9 mm, vias 2 -> 4
- net Net-(Q1-G): track 2.43 -> 5.19 mm
- net Net-(Q2-G): track 2.38 -> 5.11 mm
- net Net-(D9-A): track 0.00 -> 2.50 mm
- net Net-(D10-A): track 0.00 -> 2.02 mm
- net /USB_VBUS: track 60.6 -> 62.1 mm
- net Net-(D6-A): track 19.7 -> 20.9 mm
- net Net-(D4-A): track 23.0 -> 22.1 mm
- net Net-(SW2-A): track 15.2 -> 16.1 mm
- net Net-(D7-A): track 19.2 -> 19.9 mm, vias 3 -> 0
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Other:
- board text added: "Rev. 0.2 - © 2023 Thilo-Alexander Ginkel"
- board text removed: "Rev. 0.1 - © 2023 Thilo-Alexander Ginkel"
