File: irrigation.kicad_pcb (KiCad board)
At the start: 2 copper layers, 57.3 x 46.3 mm, 50 parts, among them J1 - 12V +, J2 - Pump 1 +, J3 - Pump 2 +, J4 USB_C_Receptacle_USB2.0, J5 Water Level, Q1 IRF7401, Q2 IRF7401, SW1 Reset, SW2 Boot, U1 TPS5430DDA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

Commit message: Add BOM, fix nets
Parts:
- C6, C8: value 100n -> 100nF
- C7: value 1u -> 1uF
- C9: value 10u -> 10uF
- D4: value 1N4148 -> B5819W SL
Connections:
- J4 pad 0: GND -> (no net)
- J4 pad 1: GND -> (no net)
- J4 pad 2: GND -> (no net)
- J4 pad 3: GND -> (no net)
Other:
- board text added: "Rev. 0.3 - © 2023-2024 Thilo-Alexander Ginkel"
- board text removed: "Rev. 0.2 - © 2023 Thilo-Alexander Ginkel"
