File: irrigation.kicad_sch (KiCad schematic)
At the start: 43 parts, among them J1 - 12V +, J2 + Pump 1 -, J3 + Pump 2 -, J3 USB_C_Receptacle_USB2.0, J5 Water Level, Q1 IRF7401, Q2 IRF7401, SW1 Boot, SW1 Reset, U1 TPS5430DDA, U2 AMS1117-3.3, U4 ESP32-C3-WROOM-02, U5 SRV05-4

Commit message: Various bug fixes & improvements
Parts:
- added D6, D7: LED, LED_SMD:LED_0603_1608Metric, symbol Device:LED
- added R3, R6: 1k, Resistor_SMD:R_0603_1608Metric, symbol Device:R
- added R4, R5: 47k, Resistor_SMD:R_0603_1608Metric, symbol Device:R
- added R9: 10k, Resistor_SMD:R_0603_1608Metric, symbol Device:R
- C9: footprint Capacitor_SMD:CP_Elec_5x5.8 -> Capacitor_SMD:CP_Elec_6.3x7.7
- J1: value - 12V + -> - 12V +
- J2: value + Pump 1 - -> - Pump 1 +
- J3: value + Pump 2 - -> - Pump 2 +
- U4: footprint Espressif:ESP32-C3-WROOM-02 -> PCM_Espressif:ESP32-C3-WROOM-02
- renumbered D8 to D10, D6 to D8, D7 to D9, R3 to R10, R4 to R11, R7 to R12, R8 to R13, R9 to R14, R5 to R7, R6 to R8
Connections:
- net GND: now also D6.1 (K), D7.1 (K), R4.2, R5.2, R9.2; no longer SW1.1, SW1.2
- net GPIO5: now also R3.1
- net GPIO6: now also R6.1
- net at Q1.4 (G), R10.2: now also R4.1
- net at Q2.4 (G), R11.2: now also R5.1
- new net: D6.2 (A), R3.2
- new net: D7.2 (A), R6.2
- new net: R9.1, SW1.1, SW1.2
Other:
- moved on the sheet: C6, R10, R11, SW1
