File: irrigation.kicad_sch (KiCad schematic)
At the start: 50 parts, among them J1 - 12V +, J2 - Pump 1 +, J3 - Pump 2 +, J3 USB_C_Receptacle_USB2.0, J5 Water Level, Q1 IRF7401, Q2 IRF7401, SW1 Boot, SW1 Reset, U1 TPS5430DDA, U2 AMS1117-3.3, U4 ESP32-C3-WROOM-02, U5 SRV05-4

Commit message: Add BOM, fix nets
Parts:
- C28: LCSC Part C15849 -> C89632
- C29: LCSC Part C15849 -> C336204
- C6, C8: value 100n -> 100nF; LCSC Part (none) -> C1591
- C7: value 1u -> 1uF; LCSC Part (none) -> C15849
- C9: value 10u -> 10uF
- D10: LCSC Part (none) -> C384865
- D2: LCSC Part (none) -> C110044
- D4: value 1N4148 -> B5819W SL; LCSC Part (none) -> C8598
- D6, D7: LCSC Part (none) -> C434419
- D8, D9: LCSC Part (none) -> C2904059
- J5: LCSC Part (none) -> C918120
- Q1, Q2: LCSC Part (none) -> C5346818
- R10, R11: LCSC Part (none) -> C22775
- R12, R14: LCSC Part (none) -> C863706
- R3: LCSC Part (none) -> C23071
- R3, R6: LCSC Part (none) -> C21190
- R4, R5: LCSC Part (none) -> C25819
- R7, R8, R9: LCSC Part (none) -> C25804
- U2: LCSC Part (none) -> C347222
Connections:
- net +5V is gone; now on net +3V3: C8.1, C9.1, C9.1, L1.2, R13.2, R4.1, R7.1, R8.1, U4.1 (3V3)
- net GND2 is gone; now on net GND: C2.2, C9.2, D1.2 (A), D2.1 (A1), D6.1 (K), D7.1 (K), J1.2 (Pin_2), Q1.1 (S), Q1.2 (S), Q1.3 (S), Q2.1 (S), Q2.2 (S), Q2.3 (S), R3.1, R4.2, R5.2, U1.6 (GND), U1.9 (GNDPAD)
- net +24V renamed +12V
